Commit message: Refactor package name from husarion_components_description to components_description
- Updated package name in CMakeLists.txt, package.xml, and README.md.
- Changed references in launch files and URDF/XACRO files to reflect the new package name.
- Modified GitHub Actions workflow to use the new package name.
- Updated changelog to reflect the new package name and maintain issue links.
- Removed obsolete environment hook file and added a new one for the updated package.

File: test/component.urdf.xacro (robot description, xacro)
@@ -5,5 +5,5 @@
   <xacro:property name="components_config_path_property" value="$(arg components_config_path)" />
   <xacro:if value="${components_config_path_property != ''}">
-    <xacro:include filename="$(find husarion_components_description)/urdf/components.urdf.xacro" ns="husarion_components" />
+    <xacro:include filename="$(find components_description)/urdf/components.urdf.xacro" ns="husarion_components" />
     <xacro:husarion_components.create_components
       components_config_path="${components_config_path_property}"

File: urdf/components.urdf.xacro (robot description, xacro)
@@ -47,5 +47,5 @@
       <xacro:if value="${type in dev_models_dict}">
         <xacro:include
-          filename="$(find husarion_components_description)/urdf/dev.urdf.xacro"
+          filename="$(find components_description)/urdf/dev.urdf.xacro"
           ns="dev"
         />
@@ -61,5 +61,5 @@
         <xacro:if value="${type == 'ANT02'}">
           <xacro:include
-            filename="$(find husarion_components_description)/urdf/teltonika_003R-00253.urdf.xacro"
+            filename="$(find components_description)/urdf/teltonika_003R-00253.urdf.xacro"
             ns="teltonika" />
           <xacro:teltonika.teltonika_003R-00253
@@ -73,5 +73,5 @@
         <xacro:if value="${type == 'CAM01'}">
           <xacro:include
-            filename="$(find husarion_components_description)/urdf/orbbec_astra.urdf.xacro"
+            filename="$(find components_description)/urdf/orbbec_astra.urdf.xacro"
             ns="camera" />
           <xacro:camera.orbbec_astra
@@ -85,5 +85,5 @@
         <xacro:if value="${type == 'CAM02'}">
           <xacro:include
-            filename="$(find husarion_components_description)/urdf/intel_realsense_d435.urdf.xacro"
+            filename="$(find components_description)/urdf/intel_realsense_d435.urdf.xacro"
             ns="camera" />
           <xacro:camera.intel_realsense_d435
@@ -105,5 +105,5 @@
           <xacro:if value="${type in zed_models_dict}">
           <xacro:include
-            filename="$(find husarion_components_description)/urdf/stereolabs_zed.urdf.xacro"
+            filename="$(find components_description)/urdf/stereolabs_zed.urdf.xacro"
             ns="camera" />
           <xacro:camera.zed_camera
@@ -123,5 +123,5 @@
         <xacro:if value="${type in luxonis_models_dict}">
           <xacro:include
-            filename="$(find husarion_components_description)/urdf/luxonis_depthai.urdf.xacro"
+            filename="$(find components_description)/urdf/luxonis_depthai.urdf.xacro"
             ns="camera" />
           <xacro:camera.luxonis_depthai
@@ -144,5 +144,5 @@
         <xacro:if value="${type in rplidar_models_dict}">
           <xacro:include
-            filename="$(find husarion_components_description)/urdf/slamtec_rplidar.urdf.xacro"
+            filename="$(find components_description)/urdf/slamtec_rplidar.urdf.xacro"
             ns="lidar"
           />
@@ -167,5 +167,5 @@
         <xacro:if value="${type in ouster_models_dict}">
           <xacro:include
-            filename="$(find husarion_components_description)/urdf/ouster.urdf.xacro"
+            filename="$(find components_description)/urdf/ouster.urdf.xacro"
             ns="lidar"
           />
@@ -181,5 +181,5 @@
         <xacro:if value="${type == 'LDR20'}">
           <xacro:include
-            filename="$(find husarion_components_description)/urdf/velodyne_puck.urdf.xacro"
+            filename="$(find components_description)/urdf/velodyne_puck.urdf.xacro"
             ns="lidar"
           />
@@ -194,5 +194,5 @@
         <xacro:if value="${type == 'MAN01'}">
           <xacro:include
-            filename="$(find husarion_components_description)/urdf/ur.urdf.xacro"
+            filename="$(find components_description)/urdf/ur.urdf.xacro"
             ns="manipulator"
           />
@@ -207,5 +207,5 @@
         <xacro:if value="${type == 'MAN02'}">
           <xacro:include
-            filename="$(find husarion_components_description)/urdf/ur.urdf.xacro"
+            filename="$(find components_description)/urdf/ur.urdf.xacro"
             ns="manipulator"
           />
@@ -220,5 +220,5 @@
         <xacro:if value="${type == 'MAN04'}">
           <xacro:include
-            filename="$(find husarion_components_description)/urdf/kinova.urdf.xacro"
+            filename="$(find components_description)/urdf/kinova.urdf.xacro"
             ns="manipulator"
           />
@@ -237,5 +237,5 @@
         <xacro:if value="${type == 'MAN05'}">
           <xacro:include
-            filename="$(find husarion_components_description)/urdf/kinova.urdf.xacro"
+            filename="$(find components_description)/urdf/kinova.urdf.xacro"
             ns="manipulator"
           />
@@ -254,5 +254,5 @@
         <xacro:if value="${type == 'MAN06'}">
           <xacro:include
-            filename="$(find husarion_components_description)/urdf/kinova.urdf.xacro"
+            filename="$(find components_description)/urdf/kinova.urdf.xacro"
             ns="manipulator"
           />
@@ -271,5 +271,5 @@
         <xacro:if value="${type == 'MAN07'}">
           <xacro:include
-            filename="$(find husarion_components_description)/urdf/kinova.urdf.xacro"
+            filename="$(find components_description)/urdf/kinova.urdf.xacro"
             ns="manipulator"
           />
@@ -287,5 +287,5 @@
         </xacro:if>
         <xacro:if value="${type == 'GRP02'}">
-          <xacro:include filename="$(find husarion_components_description)/urdf/robotiq.urdf.xacro"
+          <xacro:include filename="$(find components_description)/urdf/robotiq.urdf.xacro"
             ns="gripper" />
           <xacro:gripper.robotiq
@@ -299,5 +299,5 @@
         <xacro:if value="${type == 'WCH01'}">
           <xacro:include
-            filename="$(find husarion_components_description)/urdf/wibotic_receiver.urdf.xacro"
+            filename="$(find components_description)/urdf/wibotic_receiver.urdf.xacro"
             ns="wireless_charger" />
           <xacro:wireless_charger.wibotic_receiver

File: urdf/dev.urdf.xacro (robot description, xacro)
@@ -106,5 +106,5 @@
         <origin xyz="0 0 0" rpy="0 0 0" />
         <geometry>
-          <mesh filename="package://husarion_components_description/meshes/devs/${model}.dae"/>
+          <mesh filename="package://components_description/meshes/devs/${model}.dae"/>
         </geometry>
       </visual>

File: urdf/intel_realsense_d435.urdf.xacro (robot description, xacro)
@@ -136,5 +136,5 @@
       <link name="${component_name_underscore}color_optical_frame" />
     </xacro:if>
-    <xacro:include filename="$(find husarion_components_description)/urdf/gz_sensor.urdf.xacro" ns="gz_sensor" />
+    <xacro:include filename="$(find components_description)/urdf/gz_sensor.urdf.xacro" ns="gz_sensor" />
     <!-- It is also possible to use single rgbd_camera sensor, but using separate rgb and depth camera
       should be more accurate for D435 - different frames and fovs can be set -->

File: urdf/luxonis_depthai.urdf.xacro (robot description, xacro)
@@ -35,5 +35,5 @@
       cam_roll="${rpy.split()[0]}" cam_pitch="${rpy.split()[1]}" cam_yaw="${rpy.split()[2]}"
       simulation="${use_sim}" />
-    <xacro:include filename="$(find husarion_components_description)/urdf/gz_sensor.urdf.xacro"
+    <xacro:include filename="$(find components_description)/urdf/gz_sensor.urdf.xacro"
       ns="gz_sensor" />
     <xacro:gz_sensor.camera

File: urdf/orbbec_astra.urdf.xacro (robot description, xacro)
@@ -40,5 +40,5 @@
         <origin xyz="0.0 0.0 0.0" rpy="0.0 0.0 0.0" />
         <geometry>
-          <mesh filename="package://husarion_components_description/meshes/orbbec_astra.dae" />
+          <mesh filename="package://components_description/meshes/orbbec_astra.dae" />
         </geometry>
       </visual> -->
@@ -110,5 +110,5 @@
     <!-- GAZEBO -->
     <!-- https://github.com/orbbec/OrbbecSDK_ROS2#all-available-topics -->
-    <xacro:include filename="$(find husarion_components_description)/urdf/gz_sensor.urdf.xacro" ns="gz_sensor" />
+    <xacro:include filename="$(find components_description)/urdf/gz_sensor.urdf.xacro" ns="gz_sensor" />
     <xacro:gz_sensor.camera
       reference="${component_name_underscore}link"

File: urdf/ouster.urdf.xacro (robot description, xacro)
@@ -74,5 +74,5 @@
         <origin xyz="0.0 0.0 0.0" rpy="0.0 0.0 0.0" />
         <geometry>
-          <mesh filename="package://husarion_components_description/meshes/${mesh}.dae" />
+          <mesh filename="package://components_description/meshes/${mesh}.dae" />
         </geometry>
       </visual> -->

File: urdf/slamtec_rplidar.urdf.xacro (robot description, xacro)
@@ -211,5 +211,5 @@
         <origin xyz="0.0 0.0 0.0" rpy="0.0 0.0 0.0" />
         <geometry>
-          <mesh filename="package://husarion_components_description/meshes/rplidar/${mesh}" />
+          <mesh filename="package://components_description/meshes/rplidar/${mesh}" />
         </geometry>
       </visual> -->

File: urdf/stereolabs_zed.urdf.xacro (robot description, xacro)
@@ -305,5 +305,5 @@
     </xacro:if>
     <!-- GAZEBO -->
-    <xacro:include filename="$(find husarion_components_description)/urdf/gz_sensor.urdf.xacro" ns="gz_sensor" />
+    <xacro:include filename="$(find components_description)/urdf/gz_sensor.urdf.xacro" ns="gz_sensor" />
     <xacro:gz_sensor.camera
       reference="${component_name_underscore}camera_center"

File: urdf/teltonika_003R-00253.urdf.xacro (robot description, xacro)
@@ -35,5 +35,5 @@
         <origin xyz="0.0 0.0 0.0" rpy="0.0 0.0 0.0" />
         <geometry>
-          <mesh filename="package://husarion_components_description/meshes/teltonika_003R-00253.dae" />
+          <mesh filename="package://components_description/meshes/teltonika_003R-00253.dae" />
         </geometry>
       </visual>
@@ -42,5 +42,5 @@
         <geometry>
           <mesh
-            filename="package://husarion_components_description/meshes/teltonika_003R-00253_collision.stl" />
+            filename="package://components_description/meshes/teltonika_003R-00253_collision.stl" />
         </geometry>
       </collision>

File: urdf/ur.urdf.xacro (robot description, xacro)
@@ -58,5 +58,5 @@
       value="$(find ur_description)/config/${ur_type}/visual_parameters.yaml" scope="parent" />
     <xacro:property name="simulation_controllers"
-      value="$(find husarion_components_description)/config/ur_controllers.yaml" scope="parent" />
+      value="$(find components_description)/config/ur_controllers.yaml" scope="parent" />
       <xacro:property name="initial_positions_file" default="$(find ur_description)/config/initial_positions.yaml" />
       <xacro:property name="initial_positions"

File: urdf/velodyne_puck.urdf.xacro (robot description, xacro)
@@ -37,5 +37,5 @@
         <origin xyz="0.0 0.0 0.0" rpy="0.0 0.0 0.0" />
         <geometry>
-          <mesh filename="package://husarion_components_description/meshes/velodyne_puck.dae" />
+          <mesh filename="package://components_description/meshes/velodyne_puck.dae" />
         </geometry>
       </visual> -->

File: urdf/wibotic_receiver.urdf.xacro (robot description, xacro)
@@ -33,5 +33,5 @@
         <origin xyz="0.0 0.0 0.0" rpy="0.0 0.0 ${pi/2.0}" />
         <geometry>
-          <mesh filename="package://husarion_components_description/meshes/wibotic_receiver.stl" />
+          <mesh filename="package://components_description/meshes/wibotic_receiver.stl" />
         </geometry>
         <material name="Grey">

File: urdf/wibotic_station.urdf.xacro (robot description, xacro)
@@ -34,5 +34,5 @@
         <origin xyz="0.0 0.0 0.0" rpy="0.0 0.0 ${pi/2.0}" />
         <geometry>
-          <mesh filename="package://husarion_components_description/meshes/wibotic_station.stl" />
+          <mesh filename="package://components_description/meshes/wibotic_station.stl" />
         </geometry>
       </visual> -->
